File: Electronics/pflanzen_board/pflanzen_board.kicad_pcb (KiCad board)
At the start: 2 copper layers, 30.3 x 20.6 mm, 6 parts, among them J2 Conn_01x02_Pin, J3 Conn_01x02_Pin, J4 Conn_01x02_Pin, U1 ESP32-S3, U2 DRV8210DSGR, U3 TPS7A2501DRVR

Commit message: feat: update electronics
Parts:
- added C1: 10pF, Capacitor_SMD:C_0603_1608Metric_Pad1.08x0.95mm_HandSolder, F.Cu at (176.1, 97.9)
- added C10: 10µF, Capacitor_SMD:C_0805_2012Metric_Pad1.18x1.45mm_HandSolder, F.Cu at (188.6, 97.7)
- added C11: 10µF, Capacitor_SMD:C_0805_2012Metric_Pad1.18x1.45mm_HandSolder, F.Cu at (185.2, 84.1)
- added C12: 0.1µF, Capacitor_SMD:C_0603_1608Metric_Pad1.08x0.95mm_HandSolder, F.Cu at (183.4, 84.3)
- added C13: 220µF, Capacitor_THT:CP_Radial_D5.0mm_P2.00mm, F.Cu at (154.6, 109.8)
- added C14: 0.1µF, Capacitor_SMD:C_0603_1608Metric_Pad1.08x0.95mm_HandSolder, F.Cu at (158.4, 111.1)
- added C15: 0.1µF, Capacitor_SMD:C_0603_1608Metric_Pad1.08x0.95mm_HandSolder, F.Cu at (187.3, 112.5)
- added C16: 10µF, Capacitor_SMD:C_0805_2012Metric_Pad1.18x1.45mm_HandSolder, F.Cu at (178.7, 90.5)
- added C17: 0.1µF, Capacitor_SMD:C_0603_1608Metric_Pad1.08x0.95mm_HandSolder, F.Cu at (180.6, 90.4)
- added C2: 0.1µF, Capacitor_SMD:C_0603_1608Metric_Pad1.08x0.95mm_HandSolder, F.Cu at (182.5, 100.7)
- added C3: 0.1µF, Capacitor_SMD:C_0603_1608Metric_Pad1.08x0.95mm_HandSolder, F.Cu at (172.4, 105.3)
- added C4: 0.1µF, Capacitor_SMD:C_0603_1608Metric_Pad1.08x0.95mm_HandSolder, F.Cu at (179.4, 112.7)
- added C5: 0.1µF, Capacitor_SMD:C_0603_1608Metric_Pad1.08x0.95mm_HandSolder, F.Cu at (184.9, 112.1)
- added C6: 0.1µF, Capacitor_SMD:C_0603_1608Metric_Pad1.08x0.95mm_HandSolder, F.Cu at (176.6, 100.7)
- added C7: 0.1µF, Capacitor_SMD:C_0603_1608Metric_Pad1.08x0.95mm_HandSolder, F.Cu at (172.3, 106.9)
- added C8: 10pF, Capacitor_SMD:C_0603_1608Metric_Pad1.08x0.95mm_HandSolder, F.Cu at (182.6, 97.9)
- added C9: 1µF, Capacitor_SMD:C_0603_1608Metric_Pad1.08x0.95mm_HandSolder, F.Cu at (188.5, 99.8)
- added D1: D_TVS, Package_TO_SOT_SMD:SOT-23-6_Handsoldering, F.Cu at (180.0, 120.1)
- added D2: D_TVS, Package_TO_SOT_SMD:SOT-23-6_Handsoldering, F.Cu at (183.8, 117.1)
- added F1: Polyfuse, Fuse:Fuse_1812_4532Metric_Pad1.30x3.40mm_HandSolder, F.Cu at (195.9, 85.7)
- added J5: Conn_Coaxial, Connector_Coaxial:U.FL_Hirose_U.FL-R-SMT-1_Vertical, F.Cu at (172.9, 102.0)
- added J6: UJ20-C-H-G-SMT-1-P16-TR, Edit:USB_C_Receptacle_GCT_USB4110_Edit, F.Cu at (188.7, 124.7)
- added R1: 10kΩ, Resistor_SMD:R_0603_1608Metric_Pad0.98x0.95mm_HandSolder, F.Cu at (163.1, 97.9)
- added R10: 10kΩ, Resistor_SMD:R_0603_1608Metric_Pad0.98x0.95mm_HandSolder, F.Cu at (163.4, 113.1)
- added R11: 10kΩ, Resistor_SMD:R_0603_1608Metric_Pad0.98x0.95mm_HandSolder, F.Cu at (163.3, 114.7)
- added R12: 10kΩ, Resistor_SMD:R_0603_1608Metric_Pad0.98x0.95mm_HandSolder, F.Cu at (159.5, 117.8)
- added R13: 10kΩ, Resistor_SMD:R_0603_1608Metric_Pad0.98x0.95mm_HandSolder, F.Cu at (189.0, 112.5)
- added R14: 1kΩ, Resistor_SMD:R_0603_1608Metric_Pad0.98x0.95mm_HandSolder, F.Cu at (197.1, 114.5)
- added R15: 620Ω, Resistor_SMD:R_0603_1608Metric_Pad0.98x0.95mm_HandSolder, F.Cu at (200.8, 113.3)
- added R2: 10kΩ, Resistor_SMD:R_0603_1608Metric_Pad0.98x0.95mm_HandSolder, F.Cu at (172.4, 110.4)
- added R3: 22Ω, Resistor_SMD:R_0603_1608Metric_Pad0.98x0.95mm_HandSolder, F.Cu at (181.0, 112.7)
- added R4: 22Ω, Resistor_SMD:R_0603_1608Metric_Pad0.98x0.95mm_HandSolder, F.Cu at (182.6, 112.7)
- added R5: 10kΩ, Resistor_SMD:R_0603_1608Metric_Pad0.98x0.95mm_HandSolder, F.Cu at (181.0, 100.7)
- added R6: 10kΩ, Resistor_SMD:R_0603_1608Metric_Pad0.98x0.95mm_HandSolder, F.Cu at (179.5, 100.7)
- added R7: 10kΩ, Resistor_SMD:R_0603_1608Metric_Pad0.98x0.95mm_HandSolder, F.Cu at (172.4, 108.6)
- added R8: 10kΩ, Resistor_SMD:R_0603_1608Metric_Pad0.98x0.95mm_HandSolder, F.Cu at (197.3, 109.5)
- added R9: 10kΩ, Resistor_SMD:R_0603_1608Metric_Pad0.98x0.95mm_HandSolder, F.Cu at (197.3, 107.0)
- added SW1: SW_SPST, Button_Switch_SMD:SW_Push_1P1T_NO_6x6mm_H9.5mm, F.Cu at (165.4, 93.3)
- added SW2: SW_SPST, Button_Switch_SMD:SW_Push_1P1T_NO_6x6mm_H9.5mm, F.Cu at (165.4, 102.3)
- added U4: DRV8210DSGR, DRV8210:DRV0006A-IPC_A, F.Cu at (159.5, 114.1)
- added U5: MCP73831-5-MC, Package_DFN_QFN:DFN-8-1EP_3x2mm_P0.5mm_EP1.7x1.4mm, F.Cu at (200.2, 117.3)
- added XTAL1: NX2016SA-40M-STD-CZS-3, DRV8210:NX2016SA-40M-STD-CZS-3_NDK, F.Cu at (179.3, 97.1)
- U2: value DRV8210DSGR -> W25Q64JVSSIQ; footprint DRV8210:DRV0006A-IPC_A -> DRV8210:SOIC-8_5P28X5P28_WIN
- moved J3 72.5 mm to (200.1, 122.9), turned to 0 degrees
- moved U2 56.9 mm to (190.6, 107.7), turned to 180 degrees
- moved U3 52.0 mm to (182.7, 87.8), turned to 90 degrees
- moved J2 38.9 mm to (166.9, 107.9), turned to 0 degrees
- moved U1 38.4 mm to (180.0, 106.8)
- moved J4 32.9 mm to (153.9, 121.9)
Connections:
- net PG renamed PU
- J3 pad 1: VCC -> VBAT
- U1 pad 10: Button_1 -> unconnected-(U1-GPIO5-Pad10)
- U1 pad 11: Button_2 -> Button_1
- U1 pad 12: unconnected-(U1-GPIO7-Pad12) -> Button_2
- U1 pad 15: unconnected-(U1-GPIO10-Pad15) -> MS_1
- U1 pad 16: unconnected-(U1-GPIO11-Pad16) -> MS_2
- U1 pad 25: D- -> Net-(U1-GPIO19/USB_D-)
- U1 pad 26: D+ -> Net-(U1-GPIO20/USB_D+)
- U1 pad 30: unconnected-(U1-SPIHD-Pad30) -> HD
- U1 pad 31: unconnected-(U1-SPIWP-Pad31) -> WP
- U1 pad 32: unconnected-(U1-SPICS0-Pad32) -> CS
- U1 pad 33: unconnected-(U1-SPICLK-Pad33) -> CLK
- U1 pad 34: unconnected-(U1-SPIQ-Pad34) -> DO
- U1 pad 35: unconnected-(U1-SPID-Pad35) -> DI
- U1 pad 5: unconnected-(U1-GPIO0-Pad5) -> Net-(SW1-A)
- U1 pad 51: unconnected-(U1-GPIO45-Pad51) -> Net-(U1-GPIO45)
- U1 pad 52: unconnected-(U1-GPIO46-Pad52) -> Net-(U1-GPIO46)
- U1 pad 53: unconnected-(U1-XTAL_N-Pad53) -> XN
- U1 pad 54: unconnected-(U1-XTAL_P-Pad54) -> XP
- U1 pad 8: MS_1 -> Net-(U1-GPIO3)
- U1 pad 9: MS_2 -> unconnected-(U1-GPIO4-Pad9)
- U2 pad 1: VCC -> CS
- U2 pad 2: Motor_1 -> DO
- U2 pad 3: Motor_2 -> WP
- U2 pad 5: MS_2 -> DI
- U2 pad 6: MS_1 -> CLK
- U2 pad 7: GND -> HD
- U3 pad 7: unconnected-(U3-Thermal_Pad-Pad7) -> GND
Routing:
- net 3.3V: track 41.3 -> 136.7 mm, vias 0 -> 3
- net GND: track 19.0 -> 81.6 mm, vias 2 -> 6
- net VBAT: track 0.00 -> 46.0 mm
- net PU: track 0.00 -> 37.2 mm, vias 0 -> 2
- net VCC: track 31.5 -> 68.4 mm
- net Net-(SW1-A): track 0.00 -> 26.0 mm
- net VBUS: track 0.00 -> 21.4 mm
- net D-: track 0.00 -> 16.3 mm
- net MS_2: track 4.48 -> 19.7 mm
- net WP: track 0.00 -> 14.2 mm, vias 0 -> 2
- net CS: track 0.00 -> 13.9 mm
- net MS_1: track 4.65 -> 18.2 mm
- net D+: track 0.00 -> 13.0 mm
- net DO: track 0.00 -> 11.6 mm
- net HD: track 0.00 -> 8.46 mm
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- added copper zone on B.Cu, net GND
- added copper zone on F.Cu, net GND
Other:
- board size 30.3 x 20.6 mm -> 53.2 x 46.7 mm
- board text added: "R7"
