File: Electronics/pflanzen_board/pflanzen_board.kicad_sch (KiCad schematic)
At the start: 7 parts, among them J1 UJ20-C-H-G-SMT-1-P16-TR, J2 Conn_01x02_Pin, J3 Conn_01x02_Pin, J4 Conn_01x02_Pin, U1 ESP32-S3, U2 DRV8210DSGR, U3 TPS7A2501DRVR

Commit message: feat: update electronics
Parts:
- removed J1: UJ20-C-H-G-SMT-1-P16-TR, UJ20-C-H-G-SMT-1-P16-TR:SAMESKY_UJ20-C-H-G-SMT-1-P16-TR, symbol USB_C:UJ20-C-H-G-SMT-1-P16-TR
- added C1, C8: 10pF, Capacitor_SMD:C_0603_1608Metric_Pad1.08x0.95mm_HandSolder, symbol Device:C
- added C10, C11, C16: 10µF, Capacitor_SMD:C_0805_2012Metric_Pad1.18x1.45mm_HandSolder, symbol Device:C
- added C12, C14, C15, C17, C2, C3, C4, C5, C6, C7: 0.1µF, Capacitor_SMD:C_0603_1608Metric_Pad1.08x0.95mm_HandSolder, symbol Device:C
- added C13: 220µF, Capacitor_THT:CP_Radial_D5.0mm_P2.00mm, symbol Device:C
- added C9: 1µF, Capacitor_SMD:C_0603_1608Metric_Pad1.08x0.95mm_HandSolder, symbol Device:C
- added D1, D2: D_TVS, Package_TO_SOT_SMD:SOT-23-6_Handsoldering, symbol Device:D_TVS
- added F1: Polyfuse, Fuse:Fuse_1812_4532Metric_Pad1.30x3.40mm_HandSolder, symbol Device:Polyfuse
- added J5: Conn_Coaxial, Connector_Coaxial:U.FL_Hirose_U.FL-R-SMT-1_Vertical, symbol Connector:Conn_Coaxial
- added J6: UJ20-C-H-G-SMT-1-P16-TR, Edit:USB_C_Receptacle_GCT_USB4110_Edit, symbol Edit:UJ20-C-H-G-SMT-1-P16-TR
- added R1, R10, R11, R12, R13, R2, R5, R6, R7, R8, R9: 10kΩ, Resistor_SMD:R_0603_1608Metric_Pad0.98x0.95mm_HandSolder, symbol Device:R
- added R14: 1kΩ, Resistor_SMD:R_0603_1608Metric_Pad0.98x0.95mm_HandSolder, symbol Device:R
- added R15: 620Ω, Resistor_SMD:R_0603_1608Metric_Pad0.98x0.95mm_HandSolder, symbol Device:R
- added R3, R4: 22Ω, Resistor_SMD:R_0603_1608Metric_Pad0.98x0.95mm_HandSolder, symbol Device:R
- added SW1, SW2: SW_SPST, Button_Switch_SMD:SW_Push_1P1T_NO_6x6mm_H9.5mm, symbol Switch:SW_SPST
- added U2: W25Q64JVSSIQ, DRV8210:SOIC-8_5P28X5P28_WIN, symbol SPI:W25Q64JVSSIQ
- added U5: MCP73831-5-MC, Package_DFN_QFN:DFN-8-1EP_3x2mm_P0.5mm_EP1.7x1.4mm, symbol Battery_Management:MCP73831-5-MC
- added XTAL1: NX2016SA-40M-STD-CZS-3, DRV8210:NX2016SA-40M-STD-CZS-3_NDK, symbol Quarz:NX2016SA-40M-STD-CZS-3
- renumbered U2 to U4
Connections:
- net 3.3V: now also C10.2, C15.2, C16.2, C17.2, C2.2, C3.2, C4.2, C5.2, C6.2, C9.2, R1.2, R13.2, R2.2, R7.2, R8.2, R9.2, U2.8 (VCC)
- net ANT: now also J5.1 (In)
- net Button_1: now also U1.11 (GPIO6); no longer U1.10 (GPIO5)
- net Button_2: now also U1.12 (GPIO7); no longer U1.11 (GPIO6)
- net D+: now also D2.1 (A1), J6.A6 (DP1), J6.B6 (DP2), R4.2; no longer U1.26 (GPIO20/USB_D+)
- net D-: now also D1.1 (A1), J6.A7 (DN1), J6.B7 (DN2), R3.2; no longer U1.25 (GPIO19/USB_D-)
- net GND: now also U3.7 (Thermal_Pad), U4.9 (Thermal_Pad), C1.1, C10.1, C11.1, C12.1, C13.1, C14.1, C15.1, C16.1, C17.1, C2.1, C3.1, C4.1, C5.1, C6.1, C7.2, C8.1, C9.1, D1.2 (A2), D2.2 (A2), J6.A12_B1 (GND__1), J6.A1_B12 (GND), J6.A5 (CC1), J6.B5 (CC2), J6.SH1 (SHIELD), J6.SH2 (SHIELD__1), J6.SH3 (SHIELD__2), J6.SH4 (SHIELD__3), R10.1, R11.1, R12.1, R14.1, R5.2, R6.2, SW1.2 (B), SW2.2 (B), U2.4 (GND), U5.6 (V_{SS}), XTAL1.2, XTAL1.3; no longer U4.7 (MODE)
- net MS_1: now also U1.15 (GPIO10), R10.2; no longer U1.8 (GPIO3)
- net MS_2: now also U1.16 (GPIO11), R11.2; no longer U1.9 (GPIO4)
- net VCC: now also C11.2, C12.2, C13.2, C14.2, F1.2; no longer J3.1 (Pin_1)
- net HD: now reaches U1.30 (SPIHD)
- net HD: now also R13.1, U2.7 (/HOLD_OR_/RESET(IO3))
- net WP: now reaches U1.31 (SPIWP)
- net WP: now also R9.1, U2.3 (/WP(IO2))
- net CS: now reaches U1.32 (SPICS0)
- net CS: now also R8.1, U2.1 (/CS)
- net CLK: now reaches U1.33 (SPICLK)
- net CLK: now also U2.6 (CLK)
- net DO: now reaches U1.34 (SPIQ)
- net DO: now also U2.2 (DO(IO1))
- net DI: now reaches U1.35 (SPID)
- net DI: now also U2.5 (DI(IO0))
- net at U1.5 (GPIO0): now also R1.1, SW1.1 (A)
- net at U1.51 (GPIO45): now also R5.1
- net at U1.52 (GPIO46): now also R6.1
- net XN: now reaches U1.53 (XTAL_N)
- net XN: now also C8.2, XTAL1.1
- net XP: now reaches U1.54 (XTAL_P)
- net XP: now also C1.2, XTAL1.4
- net PG renamed PU
- net PU: now also C7.1, R7.1, SW2.1 (A)
- new net: R3.1, U1.25 (GPIO19/USB_D-)
- new net: R4.1, U1.26 (GPIO20/USB_D+)
- new net: R2.1, U1.8 (GPIO3)
- new net: R12.2, U4.7 (MODE)
- new net: R14.2, U5.8 (PROG)
- new net: R15.1, U5.5 (STAT)
- new net VBAT: F1.1, J3.1 (Pin_1), R15.2, U5.3 (V_{BAT}), U5.4 (V_{BAT})
- new net VBUS: J6.A4_B9 (VBUS), J6.A9_B4 (VBUS__1), U5.1 (V_{DD}), U5.2 (V_{DD})
- no-connect marks 46 -> 33
Other:
- note added: "ESP32-S3"
- note added: "Motor Driver"
- note added: "Oscillator"
- note added: "PinOut"
- note added: "Power Path IC"
- note added: "Power Regulator"
- note added: "SPI Flash"
- note added: "USB"
- moved on the sheet: J2, J3, J4, U1, U3, U4
